File: layout/chrono.sch (EAGLE design)
At the start: 40 parts, among them J1 22-05-7068-06, J2 22-05-7028-02, U1 TPS61016DGS, U2 STM32F100CBT6B, U3 LM293AD, U4 HC_05, X1 CRYSTALS-NOGND-4-HSMX

Commit message: routing
Parts:
- removed J2: 22-05-7028-02, con-molex:22-05-7028-02
- added R10, R11, R12, R13, R14, R15, R8, R9: (no value), rcl:R-EU_R0805
- added R16, R17, R18: 10k, rcl:R-EU_R0805
- added S1, S2: DTS-6, switch-tact:DTS-6
- added SV3: (no value), con-lstb:MA06-1
- added VT3, VT4, VT5: IRLML6402, walkgeek-eagle:IRLML6402
- J1: value 22-05-7068-06 -> 22-27-2021-02; device con-molex:22-05-7068-06 -> con-molex:22-27-2021-02
- L1: value SCD0703T-100M-N 10uH 1.44A -> SCD0703T-100M-N; device rcl:L-USL8530M -> chrono:L-US
Connections:
- removed net N$19: SV1.11
- removed net N$20: SV1.10
- removed net N$21: SV1.9
- removed net _LED_1: D1.AN, D1.AN@1
- removed net _LED_2: D2.AN, D2.AN@1
- removed net _LED_3: D3.AN, D3.AN@1
- new net A: D1.A, D2.A, D3.A, SV1.3
- new net B: D1.B, D2.B, D3.B, SV1.4
- new net B_MODE: S2.3, S2.4, U2.PA11
- new net C: D1.C, D2.C, D3.C, SV1.2
- new net D: D1.D, D2.D, D3.D, SV1.5
- new net DP: D1.DP, D2.DP, D3.DP, SV1.1
- new net E: D1.E, D2.E, D3.E, SV1.6
- new net F: D1.F, D2.F, D3.F, SV1.7
- new net G: D1.G, D2.G, D3.G, SV1.8
- new net LED_1: D1.AN, D1.AN@1, SV1.9
- new net LED_2: D2.AN, D2.AN@1, SV1.10
- new net LED_3: D3.AN, D3.AN@1, SV1.11
- new net N$10: R11.2, SV2.4
- new net N$22: R12.2, SV2.5
- new net N$23: R13.2, SV2.6
- new net N$24: R14.2, SV2.7
- new net N$25: R15.2, SV2.8
- new net N$26: SV2.9, VT4.D
- new net N$27: SV2.10, VT3.D
- new net N$28: SV2.11, VT5.D
- new net N$7: R8.2, SV2.1
- new net N$8: R9.2, SV2.2
- new net N$9: R10.2, SV2.3
- new net P_A: R10.1
- new net P_B: R11.1
- new net P_C: R9.1
- new net P_D: R12.1
- new net P_DP: R8.1
- new net P_E: R13.1
- new net P_F: R14.1
- new net P_G: R15.1
- new net P_LED1: R18.1, VT5.G
- new net P_LED2: R16.1, VT3.G
- new net P_LED3: R17.1, VT4.G
- net !NRST: now also SV3.5; no longer J1-5.S
- net +3V3: now also R16.2, R17.2, R18.2, SV3.1, U3.VCC, VT3.S, VT4.S, VT5.S; no longer J1-1.S
- net B_PWR: now also S1.3, S1.4, U2.PA10
- net GND: now also J1-2.S, S1.1, S1.2, S2.1, S2.2, SV3.3; no longer J1-3.S, J2-1.S
- net N$1: now also J1-1.S; no longer J2-2.S
- net N$11: now also U2.PB8; no longer D1.A, D2.A, D3.A
- net N$12: now also U2.PB9; no longer D1.B, D2.B, D3.B
- net N$13: now also U2.PB10; no longer D1.C, D2.C, D3.C
- net N$14: now also U2.PB11; no longer D1.D, D2.D, D3.D
- net N$15: now also U2.PB12; no longer D1.E, D2.E, D3.E
- net N$16: now also U2.PB13; no longer D1.F, D2.F, D3.F
- net N$17: now also U2.PB14; no longer D1.G, D2.G, D3.G
- net N$18: now also U2.PB15; no longer D1.DP, D2.DP, D3.DP
- net PWR_EN: now also U2.PA9
- net SWCLK: now also SV3.2; no longer J1-2.S
- net SWDIO: now also SV3.4; no longer J1-4.S
- net SWO: now also SV3.6; no longer J1-6.S
Other:
- moved on the sheet: D1, D2, D3, J1-1, J1-2, SV1, SV2

Commit message: routing
Parts:
- added R19, R20: 4.7k, rcl:R-EU_R0603
- added R21, R22: 330, rcl:R-EU_R0603
- added SV4: (no value), con-lstb:MA04-2
- C11, C12, C13, C14, C15, C16, C5, C6, C7, C8, C9: device rcl:C-EUC0805 -> rcl:C-EUC0603
- R10, R11, R12, R13, R14, R15, R16, R17, R18, R2, R3, R4, R6, R7, R8, R9: device rcl:R-EU_R0805 -> rcl:R-EU_R0603
Connections:
- new net IR1: R22.2
- new net IR2: R21.2
- new net N$21: R21.1, SV4.8
- new net N$29: R22.1, SV4.6
- net +3V3: now also R19.1, R20.1
- net GND: now also SV4.1, SV4.3, SV4.5, SV4.7
- net P_LED1: now also U2.PC15-OSC32_OUT
- net P_LED2: now also U2.PC14-OSC32_IN
- net P_LED3: now also U2.PC13-TAMPER-RTC
- net SEN_1: now also R19.2, SV4.2
- net SEN_2: now also R20.2, SV4.4
Other:
- moved on the sheet: R7, U4

Commit message: routing
Connections:
- removed net IR1: R22.2
- removed net IR2: R21.2
- removed net N$11: U2.PB8
- removed net N$12: U2.PB9
- removed net N$13: U2.PB10
- removed net N$14: U2.PB11
- removed net N$15: U2.PB12
- removed net N$16: U2.PB13
- removed net N$17: U2.PB14
- removed net N$18: U2.PB15
- new net P_IR1: R22.2, U2.PB1
- new net P_IR2: R21.2, U2.PB2
- net P_A: now also U2.PB14
- net P_B: now also U2.PB15
- net P_C: now also U2.PB13
- net P_D: now also U2.PB11
- net P_DP: now also U2.PB12
- net P_E: now also U2.PB10
- net P_F: now also U2.PB8
- net P_G: now also U2.PB9
Changed lines of the file:
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@@
 <setting verticaltext="up"/>
 </settings>
-<grid distance="0.1" unitdist="inch" unit="inch" style="lines" multiple="1" display="yes" altdistance="0.01" altunitdist="inch" altunit="inch"/>
+<grid distance="0.1" unitdist="inch" unit="inch" style="lines" multiple="1" display="no" altdistance="0.01" altunitdist="inch" altunit="inch"/>
 <layers>
 <layer number="1" name="Top" color="4" fill="1" visible="no" active="no"/>
@@
 <label x="162.56" y="-76.2" size="1.778" layer="95"/>
 </segment>
+<segment>
+<pinref part="U2" gate="A" pin="PB13"/>
+<wire x1="205.74" y1="27.94" x2="213.36" y2="27.94" width="0.1524" layer="91"/>
+<label x="208.28" y="27.94" size="1.778" layer="95"/>
+</segment>
 </net>
 <net name="P_DP" class="0">
@@
 <label x="162.56" y="-73.66" size="1.778" layer="95"/>
 </segment>
+<segment>
+<pinref part="U2" gate="A" pin="PB12"/>
+<wire x1="205.74" y1="30.48" x2="213.36" y2="30.48" width="0.1524" layer="91"/>
+<label x="208.28" y="30.48" size="1.778" layer="95"/>
+</segment>
 </net>
 <net name="P_A" class="0">
@@
 <label x="162.56" y="-78.74" size="1.778" layer="95"/>
 </segment>
+<segment>
+<pinref part="U2" gate="A" pin="PB14"/>
+<wire x1="205.74" y1="25.4" x2="213.36" y2="25.4" width="0.1524" layer="91"/>
+<label x="208.28" y="25.4" size="1.778" layer="95"/>
+</segment>
 </net>
 <net name="P_B" class="0">
@@
 <label x="162.56" y="-81.28" size="1.778" layer="95"/>
 </segment>
+<segment>
+<pinref part="U2" gate="A" pin="PB15"/>
+<wire x1="205.74" y1="22.86" x2="213.36" y2="22.86" width="0.1524" layer="91"/>
+<label x="208.28" y="22.86" size="1.778" layer="95"/>
+</segment>
 </net>
 <net name="P_D" class="0">
@@
 <label x="162.56" y="-83.82" size="1.778" layer="95"/>
 </segment>
+<segment>
+<pinref part="U2" gate="A" pin="PB11"/>
+<wire x1="205.74" y1="33.02" x2="213.36" y2="33.02" width="0.1524" layer="91"/>
+<label x="208.28" y="33.02" size="1.778" layer="95"/>
+</segment>
 </net>
 <net name="P_E" class="0">
@@
 <label x="162.56" y="-86.36" size="1.778" layer="95"/>
 </segment>
+<segment>
+<pinref part="U2" gate="A" pin="PB10"/>
+<wire x1="205.74" y1="35.56" x2="213.36" y2="35.56" width="0.1524" layer="91"/>
+<label x="208.28" y="35.56" size="1.778" layer="95"/>
+</segment>
 </net>
 <net name="P_F" class="0">
@@
 <label x="162.56" y="-88.9" size="1.778" layer="95"/>
 </segment>
+<segment>
+<pinref part="U2" gate="A" pin="PB8"/>
+<wire x1="205.74" y1="40.64" x2="213.36" y2="40.64" width="0.1524" layer="91"/>
+<label x="208.28" y="40.64" size="1.778" layer="95"/>
+</segment>
 </net>
 <net name="P_G" class="0">
@@
 <wire x1="177.8" y1="-91.44" x2="165.1" y2="-91.44" width="0.1524" layer="91"/>
 <label x="162.56" y="-91.44" size="1.778" layer="95"/>
+</segment>
+<segment>
+<pinref part="U2" gate="A" pin="PB9"/>
+<wire x1="205.74" y1="38.1" x2="213.36" y2="38.1" width="0.1524" layer="91"/>
+<label x="208.28" y="38.1" size="1.778" layer="95"/>
 </segment>
 </net>
@@
 </segment>
 </net>
-<net name="N$11" class="0">
-<segment>
-<pinref part="U2" gate="A" pin="PB8"/>
-<wire x1="205.74" y1="40.64" x2="213.36" y2="40.64" width="0.1524" layer="91"/>
-<label x="208.28" y="40.64" size="1.778" layer="95"/>
-</segment>
-</net>
-<net name="N$12" class="0">
-<segment>
-<pinref part="U2" gate="A" pin="PB9"/>
-<wire x1="205.74" y1="38.1" x2="213.36" y2="38.1" width="0.1524" layer="91"/>
-<label x="208.28" y="38.1" size="1.778" layer="95"/>
-</segment>
-</net>
-<net name="N$13" class="0">
-<segment>
-<pinref part="U2" gate="A" pin="PB10"/>
-<wire x1="205.74" y1="35.56" x2="213.36" y2="35.56" width="0.1524" layer="91"/>
-<label x="208.28" y="35.56" size="1.778" layer="95"/>
-</segment>
-</net>
-<net name="N$14" class="0">
-<segment>
-<pinref part="U2" gate="A" pin="PB11"/>
-<wire x1="205.74" y1="33.02" x2="213.36" y2="33.02" width="0.1524" layer="91"/>
-<label x="208.28" y="33.02" size="1.778" layer="95"/>
-</segment>
-</net>
-<net name="N$15" class="0">
-<segment>
-<pinref part="U2" gate="A" pin="PB12"/>
-<wire x1="205.74" y1="30.48" x2="213.36" y2="30.48" width="0.1524" layer="91"/>
-<label x="208.28" y="30.48" size="1.778" layer="95"/>
-</segment>
-</net>
-<net name="N$16" class="0">
-<segment>
-<pinref part="U2" gate="A" pin="PB13"/>
-<wire x1="205.74" y1="27.94" x2="213.36" y2="27.94" width="0.1524" layer="91"/>
-<label x="208.28" y="27.94" size="1.778" layer="95"/>
-</segment>
-</net>
-<net name="N$17" class="0">
-<segment>
-<pinref part="U2" gate="A" pin="PB14"/>
-<wire x1="205.74" y1="25.4" x2="213.36" y2="25.4" width="0.1524" layer="91"/>
-<label x="208.28" y="25.4" size="1.778" layer="95"/>
-</segment>
-</net>
-<net name="N$18" class="0">
-<segment>
-<pinref part="U2" gate="A" pin="PB15"/>
-<wire x1="205.74" y1="22.86" x2="213.36" y2="22.86" width="0.1524" layer="91"/>
-<label x="208.28" y="22.86" size="1.778" layer="95"/>
-</segment>
-</net>
 <net name="P_LED2" class="0">
 <segment>
@@
 </segment>
 </net>
-<net name="IR2" class="0">
+<net name="P_IR2" class="0">
 <segment>
 <pinref part="R21" gate="G$1" pin="2"/>
@@
 <label x="119.38" y="-15.24" size="1.778" layer="95"/>
 </segment>
-</net>
-<net name="IR1" class="0">
+<segment>
+<pinref part="U2" gate="A" pin="PB2"/>
+<wire x1="205.74" y1="55.88" x2="213.36" y2="55.88" width="0.1524" layer="91"/>
+<label x="208.28" y="55.88" size="1.778" layer="95"/>
+</segment>
+</net>
+<net name="P_IR1" class="0">
 <segment>
 <pinref part="R22" gate="G$1" pin="2"/>
@@
 <label x="129.54" y="-15.24" size="1.778" layer="95"/>
 </segment>
-</net>
+<segment>
+<pinref part="U2" gate="A" pin="PB1"/>
+<wire x1="205.74" y1="58.42" x2="213.36" y2="58.42" width="0.1524" layer="91"/>
+<label x="208.28" y="58.42" size="1.778" layer="95"/>
+</segment>
+</net>
