File: layout/chrono.brd (EAGLE design)
At the start: 99.5 x 42 mm, 40 parts, among them J1 22-05-7068-06, J2 22-05-7028-02, U1 TPS61016DGS, U2 STM32F100CBT6B, U3 LM293AD, U4 HC_05, X1 CRYSTALS-NOGND-4-HSMX

Commit message: routing
Parts:
- removed J2: 22-05-7028-02, con-molex:7395-02
- added R10, R11, R12, R13, R14, R15, R8, R9: (no value), rcl:R0805
- added R16, R17, R18: 10k, rcl:R0805
- added S1, S2: DTS-6, switch-tact:DTS-6
- added SV3: (no value), con-lstb:MA06-1
- added VT3, VT4, VT5: IRLML6402, walkgeek-eagle:MICRO3
- J1: value 22-05-7068-06 -> 22-27-2021-02; device con-molex:7395-06 -> con-molex:6410-02
- L1: value SCD0703T-100M-N 10uH 1.44A -> SCD0703T-100M-N; device rcl:L8530M -> chrono:SCD0703
- moved C16 233.2 mm to (35.6, 14.9), turned to 270 degrees
- moved C15 223.6 mm to (48.8, 15.5), turned to 180 degrees
- moved U3 221.3 mm to (39.2, 11.0), turned to 90 degrees
- moved U$1 210.7 mm to (50.1, 10.9), turned to 90 degrees
- moved R6 205.3 mm to (45.3, 31.3), turned to 90 degrees
- moved X1 200.8 mm to (45.3, 36.7), turned to 180 degrees
- moved C13 189.3 mm to (39.6, 32.3), turned to 180 degrees
- moved C12 188.6 mm to (51.4, 32.3)
- moved J1 182.2 mm to (14.1, 26.0), turned to 270 degrees
- moved R2 174.8 mm to (54.7, 21.0)
- moved C11 171.0 mm to (54.7, 23.3)
- moved C10 163.5 mm to (39.2, 30.3), turned to 180 degrees
- moved C9 161.1 mm to (42.8, 31.3), turned to 90 degrees
- moved C8 157.7 mm to (49.6, 29.6), turned to 180 degrees
- moved C7 150.7 mm to (52.0, 26.0), turned to 180 degrees
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Connections:
- removed net N$19: SV1.11
- removed net N$20: SV1.10
- removed net N$21: SV1.9
- removed net VCC: U3.8
- removed net _LED_1: D1.1, D1.6
- removed net _LED_2: D2.1, D2.6
- removed net _LED_3: D3.1, D3.6
- new net A: D1.10, D2.10, D3.10, SV1.3
- new net B: D1.9, D2.9, D3.9, SV1.4
- new net B_MODE: S2.3, S2.4, U2.32
- new net C: D1.8, D2.8, D3.8, SV1.2
- new net D: D1.5, D2.5, D3.5, SV1.5
- new net DP: D1.7, D2.7, D3.7, SV1.1
- new net E: D1.4, D2.4, D3.4, SV1.6
- new net F: D1.2, D2.2, D3.2, SV1.7
- new net G: D1.3, D2.3, D3.3, SV1.8
- new net LED_1: D1.1, D1.6, SV1.9
- new net LED_2: D2.1, D2.6, SV1.10
- new net LED_3: D3.1, D3.6, SV1.11
- new net N$10: R11.2, SV2.4
- new net N$22: R12.2, SV2.5
- new net N$23: R13.2, SV2.6
- new net N$24: R14.2, SV2.7
- new net N$25: R15.2, SV2.8
- new net N$26: SV2.9, VT4.3
- new net N$27: SV2.10, VT3.3
- new net N$28: SV2.11, VT5.3
- new net N$7: R8.2, SV2.1
- new net N$8: R9.2, SV2.2
- new net N$9: R10.2, SV2.3
- new net P_A: R10.1
- new net P_B: R11.1
- new net P_C: R9.1
- new net P_D: R12.1
- new net P_DP: R8.1
- new net P_E: R13.1
- new net P_F: R14.1
- new net P_G: R15.1
- new net P_LED1: R18.1, VT5.1
- new net P_LED2: R16.1, VT3.1
- new net P_LED3: R17.1, VT4.1
- net !NRST: now also SV3.5; no longer J1.5
- net +3V3: now also R16.2, R17.2, R18.2, SV3.1, U3.8, VT3.2, VT4.2, VT5.2; no longer J1.1
- net B_PWR: now also S1.3, S1.4, U2.31
- net GND: now also J1.2, S1.1, S1.2, S2.1, S2.2, SV3.3; no longer J1.3, J2.1
- net N$1: now also J1.1; no longer J2.2
- net N$11: now also U2.45; no longer D1.10, D2.10, D3.10
- net N$12: now also U2.46; no longer D1.9, D2.9, D3.9
- net N$13: now also U2.21; no longer D1.8, D2.8, D3.8
- net N$14: now also U2.22; no longer D1.5, D2.5, D3.5
- net N$15: now also U2.25; no longer D1.4, D2.4, D3.4
- net N$16: now also U2.26; no longer D1.2, D2.2, D3.2
- net N$17: now also U2.27; no longer D1.3, D2.3, D3.3
- net N$18: now also U2.28; no longer D1.7, D2.7, D3.7
- net N$4: now also L1.P$1; no longer L1.1
- net PWR_EN: now also U2.30
- net SWCLK: now also SV3.2; no longer J1.2
- net SWDIO: now also SV3.4; no longer J1.4
- net SWO: now also SV3.6; no longer J1.6
- net VBAT: now also L1.P$2; no longer L1.2
Routing:
- net +3V3: track 0.00 -> 79.7 mm
- net D: track 0.00 -> 37.4 mm, vias 0 -> 1
- net LED_2: track 0.00 -> 35.4 mm, vias 0 -> 1
- net E: track 0.00 -> 34.3 mm, vias 0 -> 1
- net G: track 0.00 -> 31.1 mm
- net LED_1: track 0.00 -> 30.3 mm
- net DP: track 0.00 -> 29.9 mm
- net A: track 0.00 -> 29.7 mm
- net C: track 0.00 -> 27.7 mm
- net B: track 0.00 -> 25.4 mm
- net F: track 0.00 -> 24.0 mm
- net VBAT: track 0.00 -> 22.7 mm, vias 0 -> 2
- net LED_3: track 0.00 -> 17.6 mm
- net OSC_IN: track 0.00 -> 15.7 mm
- net N$22: track 0.00 -> 14.6 mm
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- added copper zone on layer 1, net GND
Other:
- board size 99.5 x 42 mm -> 90.5 x 42 mm

Commit message: routing
Parts:
- added R19, R20: 4.7k, rcl:R0603
- added R21, R22: 330, rcl:R0603
- added SV4: (no value), con-lstb:MA04-2
- C11, C12, C13, C14, C15, C16, C5, C6, C7, C8, C9: device rcl:C0805 -> rcl:C0603
- R10, R11, R12, R13, R14, R15, R16, R17, R18, R2, R3, R4, R6, R7, R8, R9: device rcl:R0805 -> rcl:R0603
- moved R7 224.9 mm to (24.6, 4.50), turned to 180 degrees
- moved C14 191.0 mm to (32.5, 5.00), turned to 180 degrees
- moved R2 15.5 mm to (43.9, 32.1), turned to 90 degrees
- moved C11 12.2 mm to (46.3, 32.1), turned to 90 degrees
- moved C16 4.91 mm to (35.9, 10.0), turned to 0 degrees
- moved R6 3.40 mm to (48.6, 32.1)
- moved C15 2.86 mm to (51.6, 14.9)
- moved R4 2.82 mm to (39.0, 24.6)
- moved R3 2.82 mm to (36.9, 24.7)
- moved U3 2.72 mm to (39.5, 13.7), turned to 180 degrees
- moved C9 2.66 mm to (40.6, 29.8), turned to 180 degrees
- moved C10 2.50 mm to (39.9, 27.9)
- moved U$1 2.35 mm to (52.4, 10.4)
- moved C8 2.20 mm to (51.0, 27.9)
- moved C13 1.71 mm to (41.2, 32.9)
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Connections:
- new net IR1: R22.2
- new net IR2: R21.2
- new net N$21: R21.1, SV4.8
- new net N$29: R22.1, SV4.6
- net +3V3: now also R19.1, R20.1
- net GND: now also SV4.1, SV4.3, SV4.5, SV4.7
- net P_LED1: now also U2.4
- net P_LED2: now also U2.3
- net P_LED3: now also U2.2
- net SEN_1: now also R19.2, SV4.2
- net SEN_2: now also R20.2, SV4.4
Routing:
- net +3V3: track 79.7 -> 195.3 mm
- net P_LED1: track 1.80 -> 16.3 mm
- net P_LED2: track 1.80 -> 14.3 mm
- net P_LED3: track 1.80 -> 13.4 mm
- net !NRST: track 0.00 -> 7.03 mm
- net GND: track 10.2 -> 14.9 mm, vias 0 -> 2
- net OSC_IN: track 15.7 -> 11.8 mm
- net OSC_OUT: track 2.52 -> 5.02 mm

Commit message: routing
Parts:
- moved C6 1.36 mm to (50.7, 18.7)
- moved U$1 1.30 mm to (52.9, 11.6)
- moved C7 1.28 mm to (53.8, 25.8), turned to 180 degrees
- moved C15 1.12 mm to (51.4, 16.0)
- moved U3 0.57 mm to (39.9, 13.3)
- moved R19 0.50 mm to (41.4, 7.50)
- moved R20 0.50 mm to (43.5, 7.50)
- moved R21 0.50 mm to (48.7, 7.50)
- moved C16 0.22 mm to (36.0, 10.2)
- moved R3 0.10 mm to (36.8, 24.7)
- moved R4 0.10 mm to (38.9, 24.6)
Connections:
- removed net IR1: R22.2
- removed net IR2: R21.2
- removed net N$11: U2.45
- removed net N$12: U2.46
- removed net N$13: U2.21
- removed net N$14: U2.22
- removed net N$15: U2.25
- removed net N$16: U2.26
- removed net N$17: U2.27
- removed net N$18: U2.28
- new net P_IR1: R22.2, U2.19
- new net P_IR2: R21.2, U2.20
- net P_A: now also U2.27
- net P_B: now also U2.28
- net P_C: now also U2.26
- net P_D: now also U2.22
- net P_DP: now also U2.25
- net P_E: now also U2.21
- net P_F: now also U2.45
- net P_G: now also U2.46
Routing:
- net B_PWR: track 6.50 -> 59.2 mm, vias 0 -> 2
- net SEN_2: track 0.00 -> 45.4 mm, vias 0 -> 2
- net SEN_1: track 0.00 -> 44.7 mm, vias 0 -> 2
- net BT_TX: track 0.00 -> 42.8 mm, vias 0 -> 2
- net BT_RX: track 0.00 -> 41.5 mm, vias 0 -> 2
- net PWR_EN: track 0.00 -> 36.6 mm, vias 0 -> 2
- net !BT_RST: track 0.00 -> 32.4 mm, vias 0 -> 2
- net P_DP: track 0.00 -> 23.2 mm
- net P_C: track 0.00 -> 20.9 mm
- net P_D: track 0.00 -> 20.6 mm, vias 0 -> 2
- net DAC_2: track 0.00 -> 20.2 mm, vias 0 -> 2
- net P_E: track 0.00 -> 20.1 mm, vias 0 -> 2
- net GATE_2: track 0.00 -> 20.0 mm, vias 0 -> 2
- net P_IR2: track 0.00 -> 19.8 mm, vias 0 -> 2
- net GND: track 14.9 -> 34.3 mm, vias 2 -> 5
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
Commit message: routing finished
Parts:
- moved D1 18.6 mm to (81.7, 28.6), turned to 90 degrees
- moved D3 18.6 mm to (81.7, 13.4), turned to 90 degrees
- moved D2 10.7 mm to (81.7, 21.0), turned to 90 degrees
- moved SV1 5.90 mm to (89.7, 19.7), turned to 270 degrees
- moved C14 1.75 mm to (34.2, 5.40)
- moved SV3 0.40 mm to (33.6, 2.50)
Routing:
- net GND: track 34.3 -> 71.6 mm, vias 5 -> 51
- net SWCLK: track 15.1 -> 50.4 mm, vias 1 -> 2
- net !NRST: track 7.04 -> 40.4 mm, vias 0 -> 1
- net SWDIO: track 0.00 -> 30.7 mm, vias 0 -> 1
- net B_MODE: track 6.50 -> 31.7 mm, vias 0 -> 1
- net SWO: track 5.97 -> 27.9 mm
- net VBAT: track 22.7 -> 34.3 mm, vias 2 -> 4
- net PWR_EN: track 36.6 -> 39.4 mm
- net +3V3: track 207.9 -> 209.6 mm
- net N$24: track 11.9 -> 12.5 mm
- added copper zone on layer 16, net GND
Other:
- board size 90.5 x 42 mm -> 85.1 x 42 mm
